File: kicad/antenna-tuner.kicad_sch (KiCad schematic)
At the start: 0 parts

Commit message: Partial kicad schematic
Parts:
- added A1: Pololu_Breakout_A4988, Module:Pololu_Breakout-16_15.2x20.3mm, symbol Driver_Motor:Pololu_Breakout_A4988
- added C1: 100uF, symbol Device:C_Polarized
- added M1: Stepper_Motor_bipolar, symbol Motor:Stepper_Motor_bipolar
- added R1, R2, R3: 100k, symbol Device:R
- added SW1: RIGHT_FINE, symbol Switch:SW_SPST
- added SW2: RIGHT_COARSE, symbol Switch:SW_SPST
- added SW3: LEFT_COARSE, symbol Switch:SW_SPST
- added SW4: LEFT_FINE, symbol Switch:SW_SPST
Connections:
- new net: A1.13 (~{RESET}), R3.2
- new net: A1.14 (~{SLEEP}), R2.2
- new net: A1.3 (1B), M1.2 (-)
- new net: A1.4 (1A), M1.1
- new net: A1.5 (2A), M1.3
- new net: A1.6 (2B), M1.4
- new net: A1.9 (~{ENABLE}), R1.2
- new net 12V: A1.8 (VMOT), C1.1
- new net GND: A1.1 (GND), C1.2, R1.1, R2.1, R3.1, SW1.1 (A), SW2.1 (A), SW3.1 (A), SW4.1 (A)
- new net TINY_3 (PD5): A1.15 (STEP)
- new net TINY_4 (PD6): A1.16 (DIR)
- new net TINY_5V: A1.2 (VDD)
- new net TINY_A2 (PC2): SW1.2 (B)
- new net TINY_A4 (PC3): SW2.2 (B)
- new net TINY_A4 (PC4): SW3.2 (B)
- new net TINY_A5 (PC5): SW4.2 (B)
- no-connect marks 0 -> 1
Other:
- note added: "Built-in pull-up resistors"
- note added: "Step-down module"

Commit message: Updated schematic
Parts:
- added R4, R5, R7, R8: 100k, symbol Device:R
- added R6: 220, symbol Device:R
- added R9: 10k, symbol Device:R
- added U1: TCST1103, TCRT1010_VIS, symbol 2024-12-14_18-26-05:TCST1103
Connections:
- net GND: no longer A1.1 (GND), R2.1, R3.1
- net TINY_5V: now also R2.1, R3.1, R6.2, R8.1, R9.1
- net at A1.11 (MS2): now also R8.2
- net at A1.7 (GND): now also A1.1 (GND), R7.2, U1.2
- net TINY_3 (PD5): no longer names the net of A1.15 (STEP)
- net TINY_3 (PD5): now also R4.2
- net TINY_4 (PD6): no longer names the net of A1.16 (DIR)
- net TINY_4 (PD6): now also R5.2
- new net: R6.1, U1.1
- new net: R9.2, U1.3
- new net TINY_3 (PD3): R4.1
- new net TINY_4 (PD4): R5.1
- new net TINY_5 (PD5): R7.1, U1.4
Other:
- moved on the sheet: A1, R2, R3

Commit message: Added pull-ups to MS* pins. Disabled setting of microstep.
Parts:
- added R6, R8: 10k, symbol Device:R
- R7: renamed from R8; value 100k -> 10k
- renumbered R3 to R1, R9 to R10, R6 to R11, R1 to R3, R7 to R9, SW4 to SW1, SW3 to SW2, SW2 to SW3, SW1 to SW4
Connections:
- net TINY_5V: now also R6.1, R8.1
- net at A1.10 (MS1): now also R6.2
- net at A1.12 (MS3): now also R8.2
Changed lines of the file:
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@@
 	(paper "A4")
+	(junction
+		(at 59.69 74.93)
+		(diameter 0)
+		(color 0 0 0 0)
+	)
 	(junction
 		(at 59.69 59.69)
@@
 	)
 	(junction
+		(at 59.69 80.01)
+		(diameter 0)
+		(color 0 0 0 0)
+	)
+	(junction
 		(at 88.9 125.73)
 		(diameter 0)
@@
 	(wire
 		(pts
-			(xy 59.69 77.47) (xy 59.69 95.25)
+			(xy 59.69 77.47) (xy 59.69 80.01)
 		)
 		(stroke
@@
 	(wire
 		(pts
+			(xy 69.85 80.01) (xy 78.74 80.01)
+		)
+		(stroke
+			(width 0)
+			(type default)
+		)
+	)
+	(wire
+		(pts
 			(xy 63.5 114.3) (xy 50.8 114.3)
 		)
@@
 	(wire
 		(pts
+			(xy 59.69 80.01) (xy 59.69 95.25)
+		)
+		(stroke
+			(width 0)
+			(type default)
+		)
+	)
+	(wire
+		(pts
 			(xy 76.2 77.47) (xy 78.74 77.47)
 		)
@@
 	(wire
 		(pts
+			(xy 59.69 80.01) (xy 62.23 80.01)
+		)
+		(stroke
+			(width 0)
+			(type default)
+		)
+	)
+	(wire
+		(pts
 			(xy 50.8 25.4) (xy 63.5 25.4)
 		)
@@
 	(wire
 		(pts
+			(xy 59.69 74.93) (xy 59.69 77.47)
+		)
+		(stroke
+			(width 0)
+			(type default)
+		)
+	)
+	(wire
+		(pts
 			(xy 45.72 157.48) (xy 63.5 157.48)
 		)
@@
 	(wire
 		(pts
+			(xy 59.69 74.93) (xy 62.23 74.93)
+		)
+		(stroke
+			(width 0)
+			(type default)
+		)
+	)
+	(wire
+		(pts
 			(xy 58.42 69.85) (xy 78.74 69.85)
 		)
@@
 	(wire
 		(pts
+			(xy 69.85 74.93) (xy 78.74 74.93)
+		)
+		(stroke
+			(width 0)
+			(type default)
+		)
+	)
+	(wire
+		(pts
 			(xy 45.72 142.24) (xy 45.72 149.86)
 		)
@@
 	(wire
 		(pts
-			(xy 59.69 59.69) (xy 59.69 77.47)
+			(xy 59.69 59.69) (xy 59.69 74.93)
 		)
 		(stroke
@@
 		(on_board yes)
 		(dnp no)
-		(property "Reference" "R8"
+		(property "Reference" "R7"
 			(at 72.39 75.184 90)
 			(effects
@@
 			)
 		)
-		(property "Value" "100k"
+		(property "Value" "10k"
 			(at 72.39 77.47 90)
 			(effects
@@
 			(project ""
 				(path "/824c13c6-8212-484a-bd8f-6cd24ce3e475"
-					(reference "R8")
+					(reference "R7")
 					(unit 1)
 				)
@@
 		(on_board yes)
 		(dnp no)
-		(property "Reference" "SW4"
+		(property "Reference" "SW1"
 			(at 68.834 131.572 0)
 			(effects
@@
 			(project "antenna-tuner"
 				(path "/824c13c6-8212-484a-bd8f-6cd24ce3e475"
-					(reference "SW4")
+					(reference "SW1")
 					(unit 1)
 				)
@@
 		(on_board yes)
 		(dnp no)
-		(property "Reference" "SW2"
+		(property "Reference" "SW3"
 			(at 68.834 146.812 0)
 			(effects
@@
 			(project "antenna-tuner"
 				(path "/824c13c6-8212-484a-bd8f-6cd24ce3e475"
-					(reference "SW2")
+					(reference "SW3")
 					(unit 1)
 				)
@@
 				(path "/824c13c6-8212-484a-bd8f-6cd24ce3e475"
 					(reference "R4")
+					(unit 1)
+				)
+			)
+		)
+	)
+	(symbol
+		(lib_id "Device:R")
+		(at 66.04 80.01 90)
+		(unit 1)
+		(exclude_from_sim no)
+		(in_bom yes)
+		(on_board yes)
+		(dnp no)
+		(property "Reference" "R8"
+			(at 66.04 82.55 90)
+			(effects
+				(font
+					(size 1.27 1.27)
+				)
+			)
+		)
+		(property "Value" "10k"
+			(at 66.04 79.756 90)
+			(effects
+				(font
+					(size 1.27 1.27)
+				)
+			)
+		)
+		(property "Footprint" ""
+			(at 66.04 81.788 90)
+			(effects
+				(font
+					(size 1.27 1.27)
+				)
+				(hide yes)
+			)
+		)
+		(property "Datasheet" "~"
+			(at 66.04 80.01 0)
+			(effects
+				(font
+					(size 1.27 1.27)
+				)
+				(hide yes)
+			)
+		)
+		(property "Description" "Resistor"
+			(at 66.04 80.01 0)
+			(effects
+				(font
+					(size 1.27 1.27)
+				)
+				(hide yes)
+			)
+		)
+		(pin "1"
+		)
+		(pin "2"
+		)
+		(instances
+			(project ""
+				(path "/824c13c6-8212-484a-bd8f-6cd24ce3e475"
+					(reference "R8")
 					(unit 1)
 				)
@@
 		(on_board yes)
 		(dnp no)
-		(property "Reference" "R6"
+		(property "Reference" "R11"
 			(at 111.76 102.108 90)
 			(effects
@@
 			(project ""
 				(path "/824c13c6-8212-484a-bd8f-6cd24ce3e475"
-					(reference "R6")
+					(reference "R11")
 					(unit 1)
 				)
@@
 		(on_board yes)
 		(dnp no)
-		(property "Reference" "SW1"
+		(property "Reference" "SW4"
 			(at 68.834 154.432 0)
 			(effects
@@
 			(project ""
 				(path "/824c13c6-8212-484a-bd8f-6cd24ce3e475"
-					(reference "SW1")
+					(reference "SW4")
 					(unit 1)
 				)
@@
 	)
 	(symbol
+		(lib_id "Device:R")
+		(at 66.04 74.93 90)
+		(unit 1)
+		(exclude_from_sim no)
+		(in_bom yes)
+		(on_board yes)
+		(dnp no)
+		(property "Reference" "R6"
+			(at 66.294 72.644 90)
+			(effects
+				(font
+					(size 1.27 1.27)
+				)
+			)
+		)
+		(property "Value" "10k"
+			(at 65.786 74.93 90)
+			(effects
+				(font
+					(size 1.27 1.27)
+				)
+			)
+		)
+		(property "Footprint" ""
+			(at 66.04 76.708 90)
+			(effects
+				(font
+					(size 1.27 1.27)
+				)
+				(hide yes)
+			)
+		)
+		(property "Datasheet" "~"
+			(at 66.04 74.93 0)
+			(effects
+				(font
+					(size 1.27 1.27)
+				)
+				(hide yes)
+			)
+		)
+		(property "Description" "Resistor"
+			(at 66.04 74.93 0)
+			(effects
+				(font
+					(size 1.27 1.27)
+				)
+				(hide yes)
+			)
+		)
+		(pin "1"
+		)
+		(pin "2"
+		)
+		(instances
+			(project ""
+				(path "/824c13c6-8212-484a-bd8f-6cd24ce3e475"
+					(reference "R6")
+					(unit 1)
+				)
+			)
+		)
+	)
+	(symbol
 		(lib_id "Switch:SW_SPST")
 		(at 68.58 142.24 0)
@@
 		(on_board yes)
 		(dnp no)
-		(property "Reference" "SW3"
+		(property "Reference" "SW2"
 			(at 68.834 139.192 0)
 			(effects
@@
 			(project "antenna-tuner"
 				(path "/824c13c6-8212-484a-bd8f-6cd24ce3e475"
-					(reference "SW3")
+					(reference "SW2")
 					(unit 1)
 				)
@@
 		(on_board yes)
 		(dnp no)
-		(property "Reference" "R9"
+		(property "Reference" "R10"
 			(at 111.76 93.218 90)
 			(effects
@@
 			(project ""
 				(path "/824c13c6-8212-484a-bd8f-6cd24ce3e475"
-					(reference "R9")
+					(reference "R10")
 					(unit 1)
 				)
@@
 		(on_board yes)
 		(dnp no)
-		(property "Reference" "R3"
+		(property "Reference" "R1"
 			(at 64.77 55.118 90)
 			(effects
@@
 			(project ""
 				(path "/824c13c6-8212-484a-bd8f-6cd24ce3e475"
-					(reference "R3")
+					(reference "R1")
 					(unit 1)
 				)
@@
 		(on_board yes)
 		(dnp no)
-		(property "Reference" "R7"
+		(property "Reference" "R9"
 			(at 72.39 88.9 90)
 			(effects
@@
 			(project ""
 				(path "/824c13c6-8212-484a-bd8f-6cd24ce3e475"
-					(reference "R7")
+					(reference "R9")
 					(unit 1)
 				)
@@
 		(on_board yes)
 		(dnp no)
-		(property "Reference" "R1"
+		(property "Reference" "R3"
 			(at 54.61 62.738 90)
 			(effects
@@
 			(project ""
 				(path "/824c13c6-8212-484a-bd8f-6cd24ce3e475"
-					(reference "R1")
+					(reference "R3")
 					(unit 1)
 				)
